Commit message: Uploading correction of mass and inertias of compass element in chest.xacro

File: raider_description/urdf/parts/chest.xacro (robot description, xacro)
@@ -216,6 +216,6 @@
       <inertial>
         <origin xyz="-68.874374e-3 6.414726e-3 134.550735e-3" rpy="0 0 0"/>
-        <mass value="200e-3"/>
-        <inertia ixx="1.5998622965e-2" ixy="2.28234406e-4" ixz="1.9697434e-5" iyy="9.471288583e-3" iyz="-2.0465348e-3" izz="2.5385537633e-2"/>
+        <mass value="85e-3"/>
+        <inertia ixx="6.79941476e-3" ixy="9.69996226e-5" ixz="8.37140945e-6" iyy="4.025297648e-3" iyz="-8.6977729e-4" izz="1.078885349e-2"/>
       </inertial>
     </link>
