Commit message: uploading correction of inertias

File: raider_description/urdf/parts/arm.xacro (robot description, xacro)
@@ -18,8 +18,8 @@
         <origin xyz="${tY*-41.306133e-3} 3.409524e-3 129.948502e-3" rpy="0 0 0"/>
         <mass value="26e-3"/>
-        <inertia ixx="11.710303909" ixy="${tY*-0.000355401}" ixz="${tY*-1.402315479}" iyy="9.349656034" iyz="0.000185333" izz="14.505300259"/>
-      </inertial>
-    </link>
-    <joint name="joint_servo_upper_arm_${lr}" type="revolute">
+        <inertia ixx="1.1710303909e-2" ixy="${tY*-3.55401e-7}" ixz="${tY*-1.402315479e-3}" iyy="9.349656034e-3" iyz="1.85333e-7" izz="1.4505300259e-2"/>
+      </inertial>
+    </link>
+    <joint name="shoulder_${lr}_lateral" type="revolute">
       <dynamics damping="0.0" friction="0.0"/>
       <limit upper="1.5" lower="-1.5" velocity="3" effort="100"/>
@@ -45,5 +45,5 @@
         <origin xyz="${tY*(-76.059296e-3)} 3.228505e-3 308.337189e-3" rpy="0 0 0"/>
         <mass value="${mass_servo}"/>
-        <inertia ixx="${mass_servo*12008673/41834.781250}" ixy="${mass_servo*tY*(-5821.5)/41834.781250}" ixz="${mass_servo*tY*-470478.40625/41834.781250}" iyy="${mass_servo*10172087/41834.781250}" iyz="${mass_servo*(-88968.78125)/41834.781250}" izz="${mass_servo*6682665/41834.781250}"/>
+        <inertia ixx="${mass_servo*12008673e-3/41834.781250}" ixy="${mass_servo*tY*(-5821.5e-3)/41834.781250}" ixz="${mass_servo*tY*-470478.40625e-3/41834.781250}" iyy="${mass_servo*10172087e-3/41834.781250}" iyz="${mass_servo*(-88968.78125e-3)/41834.781250}" izz="${mass_servo*6682665e-3/41834.781250}"/>
       </inertial>
     </link>
@@ -70,5 +70,5 @@
         <origin xyz="${tY*-45.191589e-3} 3.468790e-3 80.072578e-3" rpy="0 0 0"/>
         <mass value="4e-3"/>
-        <inertia ixx="0.590627758" ixy="${tY*0.00000015}" ixz="${tY*0.019347738}" iyy="0.251187499" iyz="0.00000012" izz="0.811914984"/>
+        <inertia ixx="5.90627758e-4" ixy="${tY*1.5e-10}" ixz="${tY*1.9347738e-5}" iyy="2.51187499e-4" iyz="1.2e-7" izz="8.11914984e-4"/>
       </inertial>
     </link>
@@ -95,5 +95,5 @@
         <origin xyz="${tY*-45.626991e-3} 3.451273e-3 75.296814e-3" rpy="0 0 0"/>
         <mass value="4e-3"/>
-        <inertia ixx="0.255461633" ixy="${tY*-0.000014093}" ixz="${tY*0.048831278}" iyy="0.588954525" iyz="-0.000159133" izz="0.809321022"/>
+        <inertia ixx="2.55461633e-4" ixy="${tY*-1.4093e-8}" ixz="${tY*4.8831278e-5}" iyy="5.88954525e-4" iyz="-1.59133e-7" izz="8.09321022e-4"/>
       </inertial>
     </link>
@@ -120,8 +120,8 @@
         <origin xyz="${tY*-48.971466e-3} 3.471508e-3 49.196182e-3" rpy="0 0 0"/>
         <mass value="${mass_servo}"/>
-        <inertia ixx="${mass_servo*10118592/41834.781250}" ixy="${mass_servo*tY*1865.812744/41834.781250}" ixz="${mass_servo*tY*-392284.406250/41834.781250}" iyy="${mass_servo*12037051/41834.781250}" iyz="${mass_servo*(-1059.934937)/41834.781250}" izz="${mass_servo*6677542/41834.781250}"/>
-      </inertial>
-    </link>
-    <joint name="joint_servo_elbow_${lr}" type="revolute">
+        <inertia ixx="${mass_servo*10118592e-3/41834.781250}" ixy="${mass_servo*tY*1865.812744e-3/41834.781250}" ixz="${mass_servo*tY*-392284.406250e-3/41834.781250}" iyy="${mass_servo*12037051e-3/41834.781250}" iyz="${mass_servo*(-1059.934937e-3)/41834.781250}" izz="${mass_servo*6677542e-3/41834.781250}"/>
+      </inertial>
+    </link>
+    <joint name="elbow_${lr}" type="revolute">
       <dynamics damping="0.0" friction="0.0"/>
       <limit upper="${2*PI/3}" lower="${-2*PI/3}" velocity="3" effort="100"/>
@@ -147,5 +147,5 @@
         <origin xyz="${tY*-52.549400e-3} 7.686087e-3 26.149841e-3" rpy="0 0 0"/>
         <mass value="15e-3"/>
-        <inertia ixx="4.397140534" ixy="${tY*0.245999243}" ixz="${tY*0.927496479}" iyy="8.263120442" iyz="-0.566498905" izz="6.876263573"/>
+        <inertia ixx="4.397140534e-3" ixy="${tY*2.45999243e-4}" ixz="${tY*9.27496479e-4}" iyy="8.263120442e-3" iyz="-5.66498905e-4" izz="6.876263573e-4"/>
       </inertial>
     </link>
@@ -172,5 +172,5 @@
         <origin xyz="${tY*-53.241585e-3} 6.205578e-3 -1.415684e-3" rpy="0 0 0"/>
         <mass value="14e-3"/>
-        <inertia ixx="3.440210914" ixy="${tY*0.018232757}" ixz="${tY*0.095159818}" iyy="4.001844032" iyz="0.207159085" izz="4.51976604"/>
+        <inertia ixx="3.440210914e-3" ixy="${tY*1.8232757e-5}" ixz="${tY*9.5159818e-5}" iyy="4.001844032e-3" iyz="2.07159085e-3" izz="4.51976604e-3"/>
       </inertial>
     </link>
@@ -197,5 +197,5 @@
         <origin xyz="${tY*-55.055099e-3} -1.675636e-3 -6.841179e-3" rpy="0 0 0"/>
         <mass value="3.5e-3"/>
-        <inertia ixx="0.084903021" ixy="${tY*0.00951706}" ixz="${tY*0.023015952}" iyy="0.338559496" iyz="0.006557898" izz="0.325236131"/>
+        <inertia ixx="8.4903021e-3" ixy="${tY*9.51706e-6}" ixz="${tY*2.3015952e-3}" iyy="3.38559496e-4" iyz="6.557898e-6" izz="3.25236131e-4"/>
       </inertial>
     </link>
@@ -221,5 +221,5 @@
         <origin xyz="${tY*-57.381317e-3} 7.527186e-3 -48.516449e-3" rpy="0 0 0"/>
         <mass value="34e-3"/>
-        <inertia ixx="13.839519597" ixy="${tY*-0.01601312}" ixz="${tY*-0.690764395}" iyy="13.107441542" iyz="-0.183076833" izz="6.004466355"/>
+        <inertia ixx="1.3839519597e-2" ixy="${tY*-1.601312e-5}" ixz="${tY*-6.90764395e-4}" iyy="1.3107441542e-2" iyz="-1.83076833e-4" izz="6.004466355e-3"/>
       </inertial>
     </link>

File: raider_description/urdf/parts/chest.xacro (robot description, xacro)
@@ -18,5 +18,5 @@
         <origin xyz="-30.867216e-3 -3.980905e-3 103.660454e-3" rpy="0 0 0"/>
         <mass value="69e-3"/>
-        <inertia ixx="68.633104082" ixy="-0.247155947" ixz="-1.001142952" iyy="111.479482676" iyz="-2.775691149" izz="106.026365641"/>
+        <inertia ixx="6.8633104082e-2" ixy="-2.47155947e-4" ixz="-1.001142952e-3" iyy="1.11479482676e-1" iyz="-2.775691149e-3" izz="1.06026365641e-1"/>
       </inertial>
     </link>
@@ -43,5 +43,5 @@
         <origin xyz="0 -51.127079e-3 258.000061e-3" rpy="0 0 0"/>
         <mass value="10e-3"/>
-        <inertia ixx="3.170596051" ixy="-0.000000784" ixz="-0000001" iyy="5.376089166" iyz="0.000012792" izz="3.687439427"/>
+        <inertia ixx="3.170596051e-3" ixy="-7.84e-10" ixz="-1e-10" iyy="5.376089166e-3" iyz="1.2792e-8" izz="3.687439427e-3"/>
       </inertial>
     </link>
@@ -68,5 +68,5 @@
         <origin xyz="-30.197001e-3 -44.700001e-3 91.440002e-3" rpy="0 0 0"/>
         <mass value="158e-3"/>
-        <inertia ixx="22109.350504618" ixy="-0.001350018" ixz="0.003879992" iyy="128618.785627577" iyz="0.037398901" izz="122602.078416133"/>
+        <inertia ixx="22.109350504618" ixy="-1.350018e-6" ixz="3.879992e-6" iyy="128.618785627577" iyz="3.7398901e-5" izz="122.602078416133"/>
       </inertial>
     </link>
@@ -101,5 +101,5 @@
         <origin xyz="-1.480880e-3 -27.624779e-3 81.529266e-3" rpy="0 0 0"/>
         <mass value="1e-3"/>
-        <inertia ixx="0.021407978" ixy="-0.000455369" ixz="0.000088787" iyy="0.050323934" iyz="0.000335926" izz="0.07141742"/>
+        <inertia ixx="2.1407978e-5" ixy="-4.55369e-7" ixz="8.8787e-8" iyy="5.0323934e-5" iyz="3.35926e-7" izz="7.141742e-5"/>
       </inertial>
     </link>
@@ -126,5 +126,6 @@
         <origin xyz="-63.315582e-3 3.302713e-3 107.129585e-3" rpy="0 0 0"/>
         <mass value="${mass_servo}"/>
-        <inertia ixx="${mass_servo*10159775/41810.292969}" ixy="${mass_servo*1955.209106/41810.292969}" ixz="${mass_servo*86846.789062/41810.292969}" iyy="${mass_servo*12035494/41810.292969}" iyz="${mass_servo*894.308777/41810.292969}" izz="${mass_servo*6634501/41810.292969}"/>
+        <inertia ixx="${mass_servo*10159775e-3/41810.292969}" ixy="${mass_servo*1955.209106e-3/41810.292969}" ixz="${mass_servo*86846.789062e-3/41810.292969}"
+			iyy="${mass_servo*12035494e-3/41810.292969}" iyz="${mass_servo*894.308777e-3/41810.292969}" izz="${mass_servo*6634501e-3/41810.292969}"/>
       </inertial>
     </link>
@@ -151,5 +152,6 @@
         <origin xyz="0.799711e-3 3.297292e-3 107.140572e-3" rpy="0 0 0"/>
         <mass value="${mass_servo}"/>
-        <inertia ixx="${mass_servo*10171655/41810.292969}" ixy="${mass_servo*1956.694946/41810.292969}" ixz="${mass_servo*-89133.1875/41810.292969}" iyy="${mass_servo*12049550/41810.292969}" iyz="${mass_servo*-898.128174 /41810.292969}" izz="${mass_servo*6641424/41810.292969}"/>
+        <inertia ixx="${mass_servo*10171655e-3/41810.292969}" ixy="${mass_servo*1956.694946e-3/41810.292969}" ixz="${mass_servo*-89133.1875e-3/41810.292969}"
+			iyy="${mass_servo*12049550e-3/41810.292969}" iyz="${mass_servo*-898.128174e-3/41810.292969}" izz="${mass_servo*6641424e-3/41810.292969}"/>
       </inertial>
     </link>
@@ -161,6 +163,4 @@
     </joint-->
   <joint name="ultrasonic_chest" type="fixed">
-      <dynamics damping="0.0" friction="0.0"/>
-      <limit upper="0" lower="0" velocity="0" effort="100"/>
       <parent link="chest_chassis"/>
       <child link="ultrasonic_sensor"/>
@@ -184,5 +184,5 @@
         <origin xyz="-28.759998e-3 27.106962e-3 106.563263e-3" rpy="0 0 0"/>
         <mass value="10e-3"/>
-        <inertia ixx="0.466992314" ixy="0.000000648" ixz="-0.000002151" iyy="2.144495716" iyz="0.006837363" izz="0.000208781"/>
+        <inertia ixx="4.66992314e-4" ixy="6.48e-10" ixz="-2.151e-9" iyy="2.144495716e-3" iyz="6.837363e-6" izz="2.08781e-7"/>
       </inertial>
     </link>
@@ -217,5 +217,5 @@
         <origin xyz="-68.874374e-3 6.414726e-3 134.550735e-3" rpy="0 0 0"/>
         <mass value="200e-3"/>
-        <inertia ixx="15.998622965" ixy="0.228234406" ixz="0.019697434" iyy="9.471288583" iyz="-0.020465348" izz="25.385537633"/>
+        <inertia ixx="1.5998622965e-2" ixy="2.28234406e-4" ixz="1.9697434e-5" iyy="9.471288583e-3" iyz="-2.0465348e-3" izz="2.5385537633e-2"/>
       </inertial>
     </link>
@@ -242,5 +242,5 @@
         <origin xyz="-30.476395e-3 -44.831921e-3 108.771057e-3" rpy="0 0 0"/>
         <mass value="35e-3"/>
-        <inertia ixx="13.155683237" ixy="-0.019818245" ixz="-0.099426146" iyy="32.373101206" iyz="0.088507484" izz="19.455722737"/>
+        <inertia ixx="1.3155683237e-2" ixy="-1.9818245e-5" ixz="-9.9426146e-5" iyy="3.2373101206e-2" iyz="8.8507484e-5" izz="1.9455722737e-2"/>
       </inertial>
     </link>
@@ -266,5 +266,5 @@
         <origin xyz="-34.425621e-3 -52.326832e-3 105.526978e-3" rpy="0 0 0"/>
         <mass value="40e-3"/>
-        <inertia ixx="10.932820677" ixy="-1.111965118" ixz="0.114190384" iyy="36.394534502" iyz="-0.011368874" izz="26.531304424"/>
+        <inertia ixx="1.0932820677e-2" ixy="-1.111965118e-3" ixz="1.14190384e-4" iyy="3.6394534502e-2" iyz="-1.1368874e-5" izz="2.6531304424e-2"/>
       </inertial>
     </link>
@@ -290,5 +290,5 @@
         <origin xyz="3.117789e-3 -38.962219e-3 305.25e-3" rpy="0 0 0"/>
         <mass value="7.5e-3"/>
-        <inertia ixx="0.449869869" ixy="0.013904256" ixz="-0.000000129" iyy="2.367011516" iyz="-0.000000652" izz="2.033599244"/>
+        <inertia ixx="4.49869869e-4" ixy="1.3904256e-5" ixz="-1.29e-10" iyy="2.367011516e-3" iyz="-6.52e-10" izz="2.033599244e-3"/>
       </inertial>
     </link>

File: raider_description/urdf/parts/head.xacro (robot description, xacro)
@@ -18,8 +18,8 @@
         <origin xyz="-34.699566e-3 6.703261e-3 139.939987e-3" rpy="0 0 0"/>
         <mass value="13.4e-3"/>
-        <inertia ixx="0.79631024" ixy="0.071080342" ixz="0.000010505" iyy="0.707342537" iyz="-0.000000896" izz="1.203373945"/>
+        <inertia ixx="7.9631024e-4" ixy="7.1080342e-4" ixz="1.0505e-8" iyy="7.07342537e-4" iyz="-8.96e-10" izz="1.203373945e-3"/>
       </inertial>
     </link>
-    <joint name="chest_head" type="revolute">
+    <joint name="neck" type="revolute">
       <dynamics damping="0.0" friction="0.0"/>
       <limit upper="0" lower="-1" velocity="3" effort="100"/>
@@ -45,5 +45,5 @@
         <origin xyz="-31.180738e-3 -2.366833e-3 164.260635e-3" rpy="0 0 0"/>
         <mass value="44e-3"/>
-        <inertia ixx="23.419764683" ixy="-0.17967725" ixz="0.136503491" iyy="17.645258196" iyz="0.830629778" izz="26.684106335"/>
+        <inertia ixx="2.3419764683e-2" ixy="-1.7967725e-4" ixz="1.36503491e-4" iyy="1.7645258196e-2" iyz="8.30629778e-4" izz="2.6684106335e-2"/>
       </inertial>
     </link>
@@ -70,5 +70,5 @@
         <origin xyz="-49.879631e-3 9.112244e-3 143.111343e-3" rpy="0 0 0"/>
         <mass value="1e-3"/>
-        <inertia ixx="0.034414067" ixy="-0.002039668" ixz="0.001999204" iyy="0.017986123" iyz="0.014190635" izz="0.01857552"/>
+        <inertia ixx="3.4414067e-5" ixy="-2.039668e-6" ixz="1.999204e-6" iyy="1.7986123e-5" iyz="1.4190635e-5" izz="1.857552e-5"/>
       </inertial>
     </link>
@@ -95,5 +95,5 @@
         <origin xyz="-31.209848e-3 19.280575e-3 167.859589e-3" rpy="0 0 0"/>
         <mass value="3e-3"/>
-        <inertia ixx="0.151655121" ixy="0.000177538" ixz="-0.001218298" iyy="0.384780168" iyz="-0.000285021" izz="0.278011012"/>
+        <inertia ixx="1.51655121e-4" ixy="1.77538e-7" ixz="-1.218298e-6" iyy="3.84780168e-4" iyz="-2.85021e-7" izz="2.78011012e-4"/>
       </inertial>
     </link>
@@ -120,5 +120,5 @@
         <origin xyz="-24.260002e-3 -35.900002e-3 161.992737e-3" rpy="0 0 0"/>
         <mass value="3e-4"/>
-        <inertia ixx="0.001401112" ixy="0.000000002" ixz="-0.00000033" iyy="0.011750281" iyz="0.000000934" izz="0.010548865"/>
+        <inertia ixx="1.401112e-6" ixy="2e-12" ixz="-3.3e-10" iyy="1.1750281e-5" iyz="9.34e-10" izz="1.0548865e-5"/>
       </inertial>
     </link>
@@ -145,5 +145,5 @@
         <origin xyz="-31.260019e-3 13.105232e-3 167.940002e-3" rpy="0 0 0"/>
         <mass value="95.3e-3"/>
-        <inertia ixx="6.166010606" ixy="-0.000004779" ixz="0.000019444" iyy="3.256684062" iyz="0.000002913" izz="6.494934716"/>
+        <inertia ixx="6.166010606e-3" ixy="-4.779e-9" ixz="1.9444e-8" iyy="3.256684062e-3" iyz="2.913e-9" izz="6.494934716e-3"/>
       </inertial>
     </link>

File: raider_description/urdf/parts/hip.xacro (robot description, xacro)
@@ -18,5 +18,5 @@
         <origin xyz="0.000005e-3 -6.968965e-3 74.913368e-3" rpy="0 0 0"/>
         <mass value="5e-3"/>
-        <inertia ixx="1.477029903" ixy="-0.000000099" ixz="0.000000796" iyy="1.164759175" iyz="-0.00047014" izz="2.628691944"/>
+        <inertia ixx="1.477029903e-3" ixy="-9.9e-11" ixz="7.96e-10" iyy="1.164759175e-3" iyz="-4.7014e-7" izz="2.628691944e-3"/>
       </inertial>
     </link>
@@ -42,5 +42,6 @@
         <origin xyz="-0.002708e-3 -12.799425e-3 57.999710e-3" rpy="0 0 0"/>
         <mass value="${mass_servo}"/>
-        <inertia ixx="${mass_servo*12049574/41834.78125}" ixy="${mass_servo*-898.065918/41834.78125}" ixz="${mass_servo*1956.940552/41834.78125}" iyy="${mass_servo*6641437/41834.78125}" iyz="${mass_servo*-89133.273438/41834.78125}" izz="${mass_servo*10171655/41834.78125}"/>
+        <inertia ixx="${mass_servo*12049574e-3/41834.78125}" ixy="${mass_servo*-898.065918e-3/41834.78125}" ixz="${mass_servo*1956.940552e-3/41834.78125}"
+			iyy="${mass_servo*6641437e-3/41834.78125}" iyz="${mass_servo*-89133.273438e-3/41834.78125}" izz="${mass_servo*10171655e-3/41834.78125}"/>
       </inertial>
     </link>
@@ -66,8 +67,8 @@
         <origin xyz="0 8.793029e-3 50.608299e-3" rpy="0 0 0"/>
         <mass value="16e-3"/>
-        <inertia ixx="5.191173851" ixy="0.000000575" ixz="-0.000000273" iyy="4.106148647" iyz="-1.012029816" izz="5.375464492"/>
+        <inertia ixx="5.191173851e-3" ixy="5.75e-10" ixz="-2.73e-10" iyy="4.106148647e-3" iyz="-1.012029816e-3" izz="5.375464492e-3"/>
       </inertial>
     </link>
-    <joint name="bracket_servo_right" type="revolute">
+    <joint name="hip_right_lateral" type="revolute">
       <dynamics damping="0.0" friction="0.0"/>
       <limit upper="${PI}" lower="${-PI}" velocity="3" effort="100"/>
@@ -103,8 +104,9 @@
         <origin xyz="-32.002708e-3 -8.200576e-3 55.880287e-3" rpy="0 0 0"/>
         <mass value="${mass_servo}"/>
-        <inertia ixx="${mass_servo*12049575/41834.78125}" ixy="${mass_servo*898.116455/41834.78125}" ixz="${mass_servo*-1957.101929/41834.78125}" iyy="${mass_servo*6641438/41834.78125}" iyz="${mass_servo*-89133.156250/41834.78125}" izz="${mass_servo*10171655/41834.78125}"/>
+        <inertia ixx="${mass_servo*12049575e-3/41834.78125}" ixy="${mass_servo*898.116455e-3/41834.78125}" ixz="${mass_servo*-1957.101929e-3/41834.78125}"
+			iyy="${mass_servo*6641438e-3/41834.78125}" iyz="${mass_servo*-89133.156250e-3/41834.78125}" izz="${mass_servo*10171655e-3/41834.78125}"/>
       </inertial>
     </link>
-    <joint name="bracket_servo_left" type="revolute">
+    <joint name="hip_left_lateral" type="revolute">
       <dynamics damping="0.0" friction="0.0"/>
       <limit upper="${PI}" lower="${-PI}" velocity="3" effort="100"/>
@@ -130,5 +132,6 @@
         <origin xyz="31.997292e-3 -8.200576e-3 55.880287e-3" rpy="0 0 0"/>
         <mass value="${mass_servo}"/>
-        <inertia ixx="${mass_servo*12049552/41834.78125}" ixy="${mass_servo*898.090698/41834.78125}" ixz="${mass_servo*-1956.938599/41834.78125}" iyy="${mass_servo*6641408.5/41834.78125}" iyz="${mass_servo*-89132.632812/41834.78125}" izz="${mass_servo*10171655/41834.78125}"/>
+        <inertia ixx="${mass_servo*12049552e-3/41834.78125}" ixy="${mass_servo*898.090698e-3/41834.78125}" ixz="${mass_servo*-1956.938599e-3/41834.78125}"
+			iyy="${mass_servo*6641408.5e-3/41834.78125}" iyz="${mass_servo*-89132.632812e-3/41834.78125}" izz="${mass_servo*10171655e-3/41834.78125}"/>
       </inertial>
     </link>
