Commit message: Deleting unnecessary lines and adding a velocity controller to try holding the robot

File: raider_description/urdf/parts/arm.xacro (robot description, xacro)
@@ -43,7 +43,7 @@
       </visual>
       <inertial>
-        <origin xyz="${tY*(-76.059296e-3)} 3.228505e-3 308.337189e-3" rpy="0 0 0"/>
+        <origin xyz="${tY*(-43.683769e-3)} 4.528502e-3 106.228104e-3" rpy="0 0 0"/>
         <mass value="${mass_servo}"/>
-        <inertia ixx="${mass_servo*12008673e-3/41834.781250}" ixy="${mass_servo*tY*(-5821.5e-3)/41834.781250}" ixz="${mass_servo*tY*-470478.40625e-3/41834.781250}" iyy="${mass_servo*10172087e-3/41834.781250}" iyz="${mass_servo*(-88968.78125e-3)/41834.781250}" izz="${mass_servo*6682665e-3/41834.781250}"/>
+        <inertia ixx="1.5841490372e-4" ixy="${tY*2.571e-6}" ixz="${tY*1.194e-6}" iyy="-2.571e-6" iyz="1.3372638e-2" izz="8.731449e-3"/>
       </inertial>
     </link>
@@ -118,7 +118,7 @@
       </visual>
       <inertial>
-        <origin xyz="${tY*-48.971466e-3} 3.471508e-3 49.196182e-3" rpy="0 0 0"/>
+        <origin xyz="${tY*-44.74e-3} 3.471498e-3 48.827362e-3" rpy="0 0 0"/>
         <mass value="${mass_servo}"/>
-        <inertia ixx="${mass_servo*10118592e-3/41834.781250}" ixy="${mass_servo*tY*1865.812744e-3/41834.781250}" ixz="${mass_servo*tY*-392284.406250e-3/41834.781250}" iyy="${mass_servo*12037051e-3/41834.781250}" iyz="${mass_servo*(-1059.934937e-3)/41834.781250}" izz="${mass_servo*6677542e-3/41834.781250}"/>
+        <inertia ixx="1.3372631e-2" ixy="${tY*2.572816e-6}" ixz="${tY*-1.17185437e-4}" iyy="1.5841492015e-2" iyz="-1.180748e-6" izz="8.73145096e-3"/>
       </inertial>
     </link>

File: raider_description/urdf/parts/chest.xacro (robot description, xacro)
@@ -66,7 +66,7 @@
       </visual>
       <inertial>
-        <origin xyz="-30.197001e-3 -44.700001e-3 91.440002e-3" rpy="0 0 0"/>
-        <mass value="158e-3"/>
-        <inertia ixx="22.109350504618" ixy="-1.350018e-6" ixz="3.879992e-6" iyy="128.618785627577" iyz="3.7398901e-5" izz="122.602078416133"/>
+        <origin xyz="1.062995e-3 -48.5e-3 56.44e-3" rpy="0 0 0"/>
+        <mass value="109e-3"/>
+        <inertia ixx="1.52527e-4" ixy="3.27e-10" ixz="-3.529795e-6" iyy="8.8730716716e-2" iyz="2.4012e-8" izz="8.4579923136e-2"/>
       </inertial>
     </link>
@@ -77,12 +77,4 @@
       <origin xyz="30.67e-3 -25.94e-3 -4e-3"/>
     </joint>
-  <!--joint name="joint_accelerometer_chest" type="revolute">
-      <dynamics damping="0.0" friction="0.0"/>
-      <limit upper="0" lower="0" velocity="0" effort="100"/>
-      <parent link="chest_chassis"/>
-      <child link="accelerometer"/>
-      <origin xyz="30.67e-3 -25.94e-3 -4e-3"/>
-      <axis xyz="0 1 0"/>
-    </joint-->
     <link name="accelerometer">
       <collision>
@@ -126,6 +118,6 @@
         <origin xyz="-63.315582e-3 3.302713e-3 107.129585e-3" rpy="0 0 0"/>
         <mass value="${mass_servo}"/>
-        <inertia ixx="${mass_servo*10159775e-3/41810.292969}" ixy="${mass_servo*1955.209106e-3/41810.292969}" ixz="${mass_servo*86846.789062e-3/41810.292969}"
-			iyy="${mass_servo*12035494e-3/41810.292969}" iyz="${mass_servo*894.308777e-3/41810.292969}" izz="${mass_servo*6634501e-3/41810.292969}"/>
+        <inertia ixx="1.3356931987e-4" ixy="2.570283e-6" ixz="1.14185394e-4"
+			iyy="1.5822969271e-4" iyz="1.176189e-6" izz="8.7223651e-3"/>
       </inertial>
     </link>
@@ -152,6 +144,6 @@
         <origin xyz="0.799711e-3 3.297292e-3 107.140572e-3" rpy="0 0 0"/>
         <mass value="${mass_servo}"/>
-        <inertia ixx="${mass_servo*10171655e-3/41810.292969}" ixy="${mass_servo*1956.694946e-3/41810.292969}" ixz="${mass_servo*-89133.1875e-3/41810.292969}"
-			iyy="${mass_servo*12049550e-3/41810.292969}" iyz="${mass_servo*-898.128174e-3/41810.292969}" izz="${mass_servo*6641424e-3/41810.292969}"/>
+        <inertia ixx="1.3356942504e-2" ixy="2.56949e-6" ixz="-1.14164863e-4"
+			iyy="1.14164863e-4" iyz="1.5822945607e-2" izz="8.722356554e-3"/>
       </inertial>
     </link>
@@ -193,12 +185,4 @@
       <origin xyz="-42.52e-3 0 58.46e-3"/>
     </joint>
-  <!--joint name="compass_chest" type="revolute">
-      <dynamics damping="0.0" friction="0.0"/>
-      <limit upper="0" lower="0" velocity="0" effort="100"/>
-      <parent link="chest_chassis"/>
-      <child link="compass"/>
-      <origin xyz="-42.52e-3 0 58.46e-3"/>
-      <axis xyz="0 1 0"/>
-    </joint-->
     <link name="compass">
       <collision>

File: raider_description/urdf/parts/hip.xacro (robot description, xacro)
@@ -42,6 +42,6 @@
         <origin xyz="-0.002708e-3 -12.799425e-3 57.999710e-3" rpy="0 0 0"/>
         <mass value="${mass_servo}"/>
-        <inertia ixx="${mass_servo*12049574e-3/41834.78125}" ixy="${mass_servo*-898.065918e-3/41834.78125}" ixz="${mass_servo*1956.940552e-3/41834.78125}"
-			iyy="${mass_servo*6641437e-3/41834.78125}" iyz="${mass_servo*-89133.273438e-3/41834.78125}" izz="${mass_servo*10171655e-3/41834.78125}"/>
+        <inertia ixx="1.582297716e-2" ixy="-1.176645e-6" ixz="2.569658e-6"
+			iyy="8.722344065e-3" iyz="-1.14167461e-4" izz="1.3356987204e-2"/>
       </inertial>
     </link>
@@ -102,8 +102,8 @@
       </visual>
       <inertial>
-        <origin xyz="-32.002708e-3 -8.200576e-3 55.880287e-3" rpy="0 0 0"/>
+        <origin xyz="-32.002712e-3 -8.189585e-3 56.084415e-3" rpy="0 0 0"/>
         <mass value="${mass_servo}"/>
-        <inertia ixx="${mass_servo*12049575e-3/41834.78125}" ixy="${mass_servo*898.116455e-3/41834.78125}" ixz="${mass_servo*-1957.101929e-3/41834.78125}"
-			iyy="${mass_servo*6641438e-3/41834.78125}" iyz="${mass_servo*-89133.156250e-3/41834.78125}" izz="${mass_servo*10171655e-3/41834.78125}"/>
+        <inertia ixx="1.5822986362e-2" ixy="1.176784e-6" ixz="-2.566336e-6"
+			iyy="8.722364442e-3" iyz="-1.1416591e-4" izz="1.3356989833e-2"/>
       </inertial>
     </link>
@@ -132,6 +132,6 @@
         <origin xyz="31.997292e-3 -8.200576e-3 55.880287e-3" rpy="0 0 0"/>
         <mass value="${mass_servo}"/>
-        <inertia ixx="${mass_servo*12049552e-3/41834.78125}" ixy="${mass_servo*898.090698e-3/41834.78125}" ixz="${mass_servo*-1956.938599e-3/41834.78125}"
-			iyy="${mass_servo*6641408.5e-3/41834.78125}" iyz="${mass_servo*-89132.632812e-3/41834.78125}" izz="${mass_servo*10171655e-3/41834.78125}"/>
+        <inertia ixx="1.5823002139e-2" ixy="1.176567e-6" ixz="-2.564784e-6"
+			iyy="8.722373645e-3" iyz="-1.14165109e-4" izz="1.3356987204e-2"/>
       </inertial>
     </link>

File: raider_description/urdf/parts/leg.xacro (robot description, xacro)
@@ -70,6 +70,6 @@
         <origin xyz="${tY*33.059711e-3} -4.057295e-3 -160.200577e-3" rpy="0 0 0"/>
         <mass value="${mass_servo}"/>
-        <inertia ixx="${mass_servo*10159.758/41810.285156}" ixy="${mass_servo*tY*(-1.954405151)/41810.285156}" ixz="${mass_servo*tY*86.83878125/41810.285156}"
-			iyy="${mass_servo*12035.474/41810.285156}" iyz="${mass_servo*(-895.013855e-3)/41810.285156}" izz="${mass_servo*6634505.5e-3/41810.285156}"/>
+        <inertia ixx="1.3372616303e-2" ixy="${tY*-2.572339e-6}" ixz="${tY*1.17188816e-4}"
+			iyy="1.5841409189e-2" iyz="-1.178714e-6" izz="8.731462792e-3"/>
       </inertial>
     </link>
@@ -119,6 +119,6 @@
         <origin xyz="${tY*31.997292e-3} -44.940292e-3 -160.200577e-3" rpy="0 0 0"/>
         <mass value="${mass_servo}"/>
-        <inertia ixx="${mass_servo*12049.5/41810.285156}" ixy="${mass_servo*tY*1.957543335/41810.285156}" ixz="${mass_servo*tY*899.625366e-3/41810.285156}"
-			iyy="${mass_servo*10171.751/41810.285156}" iyz="${mass_servo*89.138367188/41810.285156}" izz="${mass_servo*6641.419/41810.285156}"/>
+        <inertia ixx="1.5823028433e-2" ixy="${tY*2.575489e-6}" ixz="${tY*1.180097e-6}"
+			iyy="1.335689386e-2" iyz="1.14169813e-4" izz="8.722369701e-3"/>
       </inertial>
     </link>
@@ -174,6 +174,6 @@
         <origin xyz="${tY*33.059711e-3} -16.859426e-3 -97.997299e-3" rpy="0 0 0"/>
         <mass value="${mass_servo}"/>
-        <inertia ixx="${mass_servo*10159.758/41810.289062}" ixy="${mass_servo*tY*(-86.838)/41810.289062}" ixz="${mass_servo*tY*(-1.954375122)/41810.289062}"
-			iyy="${mass_servo*6634.506/41810.289062}" iyz="${mass_servo*895.015137/41810.289062}" izz="${mass_servo*12035.475/41810.289062}"/>
+        <inertia ixx="1.3356996407e-4" ixy="${tY*-1.14167133e-4}" ixz="${tY*-2.564833e-3}"
+			iyy="8.722380219e-3" iyz="1.169343e-6" izz="1.5822973216e-2"/>
       </inertial>
     </link>
@@ -218,6 +218,6 @@
         <origin xyz="${tY*14.675918e-3} -31.720392e-3 -78.538040e-3" rpy="0 0 0"/>
         <mass value="2e-3"/>
-        <inertia ixx="${(2e-3)*365.223125/1726.713501}" ixy="${tY*(2e-3)*-6.505744629/1726.713501}" ixz="${tY*(2e-3)*1.741682983/1726.713501}"
-			iyy="${(2e-3)*118.269359375/1726.713501}" iyz="${(2e-3)*58.177648438/1726.713501}" izz="${(2e-3)*250.800671875/1726.713501}"/>
+        <inertia ixx="4.23030511e-4" ixy="${tY*7.535441e-6}" ixz="${tY*-2.017274e-3}"
+			iyy="1.36991903e-4" iyz="6.7384774e-5" izz="2.90495255e-4"/>
       </inertial>
     </link>
@@ -248,6 +248,6 @@
         <origin xyz="${tY*33.059711e-3} -16.859426e-3 -65.997299e-3" rpy="0 0 0"/>
         <mass value="${mass_servo}"/>
-        <inertia ixx="${mass_servo*10171.693/41834.785156}" ixy="${mass_servo*tY*(-89.132875)/41834.785156}" ixz="${mass_servo*tY*(-1.956631226)/41834.785156}"
-			iyy="${mass_servo*6641.4265/41834.785156}" iyz="${mass_servo*898.551575e-3/41834.785156}" izz="${mass_servo*12049.564/41834.785156}"/>
+        <inertia ixx="1.3372655744e-2" ixy="${tY*-1.1718175e-4}" ixz="${tY*2.571199e-6}"
+			iyy="8.731482512e-3" iyz="1.172656e-6" izz="1.5841505162e-2"/>
       </inertial>
     </link>
@@ -301,6 +301,6 @@
         <origin xyz="${tY*33.259712e-3} -4.062710e-3 -3.799430e-3" rpy="0 0 0"/>
         <mass value="${mass_servo}"/>
-        <inertia ixx="${mass_servo*10159.758/41810.289062}" ixy="${mass_servo*tY*1.954408447/441810.289062}" ixz="${mass_servo*tY*(-86.838867188)/41810.289062}"
-			iyy="${mass_servo*12035.474/41810.289062}" iyz="${mass_servo*-895.017456e-3/41810.289062}" izz="${mass_servo*6634.506/41810.289062}"/>
+        <inertia ixx="1.3372630764e-2" ixy="${tY*2.572295e-6}" ixz="${tY*-1.17182951e-4}"
+			iyy="1.5841502533e-2" iyz="-1.180558e-6" izz="8.731446358e-3"/>
       </inertial>
     </link>
@@ -396,8 +396,8 @@
       </visual>
       <inertial>
-        <origin xyz="${tY*31.997288e-3} -37.115585e-3 -3.810416e-3" rpy="0 0 0"/>
-        <mass value="${mass_servo}"/>
-        <inertia ixx="${mass_servo*12035.472/41810.289062}" ixy="${mass_servo*tY*(-1.954408440820347)/441810.289062}" ixz="${mass_servo*tY*(-895.014343e-3)/41810.289062}"
-			iyy="${mass_servo*10159.758/41810.289062}" iyz="${mass_servo*86.838570312/41810.289062}" izz="${mass_servo*6634.5085/41810.289062}"/>
+        <origin xyz="${tY*32.002708e-3} -41.380287e-3 -3.799424e-3" rpy="0 0 0"/>
+        <mass value="${mass_servo}"/>
+        <inertia ixx="1.5841507791e-2" ixy="${tY*-2.568826e-6}" ixz="${tY*1.180211e-6}"
+			iyy="1.3372622876e-2" iyz="-1.17182284e-4" izz="8.731452274e-3"/>
       </inertial>
     </link>
